Commit message: new features for Siggraph Asia paper

File: humanSubject01/humanSubject01_48dof.urdf (robot description, URDF)
Before this commit: robot XSensStyleModel_template, 51 links, 50 joints
Links:
- removed link LeftHandCOM
- removed link RightHandCOM
Joints:
- removed joint jLeftHandCOM
- removed joint jRightHandCOM

File: humanSubject01/humanSubject01_48dof_noJointLimit.urdf (robot description, URDF)
Before this commit: robot XSensStyleModel_template, 51 links, 50 joints
Links:
- removed link LeftHandCOM
- removed link RightHandCOM
Joints:
- removed joint jLeftHandCOM
- removed joint jRightHandCOM

File: humanSubject01/humanSubject01_66dof.urdf (robot description, URDF)
Before this commit: robot XSensStyleModel_template, 69 links, 68 joints
Links:
- removed link LeftHandCOM
- removed link RightHandCOM
Joints:
- removed joint jLeftHandCOM
- removed joint jRightHandCOM

File: humanSubject01/humanSubject01_66dof_colored.urdf (robot description, URDF)
Before this commit: robot XSensStyleModel_template, 69 links, 68 joints
Links:
- removed link LeftHandCOM
- removed link RightHandCOM
Joints:
- removed joint jLeftHandCOM
- removed joint jRightHandCOM

File: humanSubject02/humanSubject02_48dof.urdf (robot description, URDF)
Before this commit: robot XSensStyleModel_template, 51 links, 50 joints
Links:
- removed link LeftHandCOM
- removed link RightHandCOM
Joints:
- removed joint jLeftHandCOM
- removed joint jRightHandCOM

File: humanSubject02/humanSubject02_48dof_noJointLimit.urdf (robot description, URDF)
Before this commit: robot XSensStyleModel_template, 51 links, 50 joints
Links:
- removed link LeftHandCOM
- removed link RightHandCOM
Joints:
- removed joint jLeftHandCOM
- removed joint jRightHandCOM

File: humanSubject03/humanSubject03_48dof.urdf (robot description, URDF)
Before this commit: robot XSensStyleModel_template, 51 links, 50 joints
Links:
- removed link LeftHandCOM
- removed link RightHandCOM
Joints:
- removed joint jLeftHandCOM
- removed joint jRightHandCOM

File: humanSubject03/humanSubject03_48dof_noJointLimit.urdf (robot description, URDF)
Before this commit: robot XSensStyleModel_template, 51 links, 50 joints
Links:
- removed link LeftHandCOM
- removed link RightHandCOM
Joints:
- removed joint jLeftHandCOM
- removed joint jRightHandCOM

File: humanSubject04/humanSubject04_48dof.urdf (robot description, URDF)
Before this commit: robot XSensStyleModel_template, 51 links, 50 joints
Links:
- removed link LeftHandCOM
- removed link RightHandCOM
Joints:
- removed joint jLeftHandCOM
- removed joint jRightHandCOM

File: humanSubject04/humanSubject04_48dof_noJointLimit.urdf (robot description, URDF)
Before this commit: robot XSensStyleModel_template, 51 links, 50 joints
Links:
- removed link LeftHandCOM
- removed link RightHandCOM
Joints:
- removed joint jLeftHandCOM
- removed joint jRightHandCOM

File: humanSubject04/humanSubject04_66dof.urdf (robot description, URDF)
Before this commit: robot XSensStyleModel_template, 69 links, 68 joints
Links:
- removed link LeftHandCOM
- removed link RightHandCOM
Joints:
- removed joint jLeftHandCOM
- removed joint jRightHandCOM

File: humanSubject05/humanSubject05_48dof.urdf (robot description, URDF)
Before this commit: robot XSensStyleModel_template, 51 links, 50 joints
Links:
- removed link LeftHandCOM
- removed link RightHandCOM
Joints:
- removed joint jLeftHandCOM
- removed joint jRightHandCOM

File: humanSubject05/humanSubject05_48dof_noJointLimit.urdf (robot description, URDF)
Before this commit: robot XSensStyleModel_template, 51 links, 50 joints
Links:
- removed link LeftHandCOM
- removed link RightHandCOM
Joints:
- removed joint jLeftHandCOM
- removed joint jRightHandCOM

File: humanSubject05/humanSubject05_66dof.urdf (robot description, URDF)
Before this commit: robot XSensStyleModel_template, 69 links, 68 joints
Links:
- removed link LeftHandCOM
- removed link RightHandCOM
Joints:
- removed joint jLeftHandCOM
- removed joint jRightHandCOM

File: humanSubject06/humanSubject06_48dof.urdf (robot description, URDF)
Before this commit: robot XSensStyleModel_template, 51 links, 50 joints
Links:
- removed link LeftHandCOM
- removed link RightHandCOM
Joints:
- removed joint jLeftHandCOM
- removed joint jRightHandCOM

File: humanSubject06/humanSubject06_48dof_noJointLimit.urdf (robot description, URDF)
Before this commit: robot XSensStyleModel_template, 51 links, 50 joints
Links:
- removed link LeftHandCOM
- removed link RightHandCOM
Joints:
- removed joint jLeftHandCOM
- removed joint jRightHandCOM

File: humanSubject06/humanSubject06_66dof.urdf (robot description, URDF)
Before this commit: robot XSensStyleModel_template, 69 links, 68 joints
Links:
- removed link LeftHandCOM
- removed link RightHandCOM
Joints:
- removed joint jLeftHandCOM
- removed joint jRightHandCOM

File: humanSubject07/humanSubject07_48dof.urdf (robot description, URDF)
Before this commit: robot XSensStyleModel_template, 51 links, 50 joints
Links:
- removed link LeftHandCOM
- removed link RightHandCOM
Joints:
- removed joint jLeftHandCOM
- removed joint jRightHandCOM

File: humanSubject07/humanSubject07_48dof_noJointLimit.urdf (robot description, URDF)
Before this commit: robot XSensStyleModel_template, 51 links, 50 joints
Links:
- removed link LeftHandCOM
- removed link RightHandCOM
Joints:
- removed joint jLeftHandCOM
- removed joint jRightHandCOM

File: humanSubject07/humanSubject07_66dof.urdf (robot description, URDF)
Before this commit: robot XSensStyleModel_template, 69 links, 68 joints
Links:
- removed link LeftHandCOM
- removed link RightHandCOM
Joints:
- removed joint jLeftHandCOM
- removed joint jRightHandCOM
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